File: MZCF-KBD01L.kicad_sch (KiCad schematic)
At the start: 114 parts, among them CN1 XH-4AW_C2908613, SW1 SW_Push, SW10 SW_Push, SW11 SW_Push, SW12 SW_Push, SW13 SW_Push, SW14 SW_Push, SW15 SW_Push, SW16 SW_Push, SW17 SW_Push, SW18 SW_Push, SW19 SW_Push, SW2 SW_Push, SW20 SW_Push, SW21 SW_Push, SW22 SW_Push, SW23 SW_Push, SW24 SW_Push, SW25 SW_Push, SW26 SW_Push, SW27 SW_Push, SW28 SW_Push, SW29 SW_Push, SW3 SW_Push, SW30 SW_Push, SW31 SW_Push, SW32 SW_Push, SW33 SW_Push, SW34 SW_Push, SW35 SW_Push, SW36 SW_Push, SW37 SW_Push, SW38 SW_Push, SW39 SW_Push, SW4 SW_Push, SW40 SW_Push, SW41 SW_Push, SW42 SW_Push, SW43 SW_Push, SW44 SW_Push, SW45 SW_Push, SW46 SW_Push, SW47 SW_Push, SW48 SW_Push, SW49 SW_Push, SW5 SW_Push, SW50 SW_Push, SW51 SW_Push, SW52 SW_Push, SW53 SW_Push, SW54 SW_Push, SW55 SW_Push, SW56 SW_Push, SW6 SW_Push, SW7 SW_Push, SW8 SW_Push, SW9 SW_Push, U1 RP2040-ZERO

Commit message: feat: new left keyboard
Parts:
- removed CN1: XH-4AW_C2908613, lcsc_footprints:C2908613_CONN-TH_XH-4AW, symbol lcsc_imported:XH-4AW_C2908613
- removed D14, D21, D28, D35, D42, D56, D7: 1N4148W, symbol Diode:1N4148W
- removed SW14, SW21, SW28, SW35, SW42, SW49, SW56, SW7: SW_Push, symbol Switch:SW_Push
- added CN1: PJ-320A_C49284721, lcsc_footprints:C49284721_AUDIO-TH_PJ-320A_C49284721, symbol lcsc_imported:PJ-320A_C49284721
- added D50, D51, D52, D53, D54: 1N4148W, symbol Diode:1N4148W
- added SW50, SW51, SW52, SW53, SW54: SW_Push, symbol Switch:SW_Push
- added SW55: EC11E1834403, lcsc_footprints:C361165_SW-TH_EC11E1820402, symbol lcsc_imported:EC11E1834403
- renumbered D11 to D10, D12 to D11, D13 to D12, D15 to D13, D16 to D14, D17 to D15, D18 to D16, D19 to D17, D20 to D18, D22 to D19, D23 to D20, D24 to D21, D25 to D22, D26 to D23, D27 to D24, D29 to D25, D30 to D26, D31 to D27, D32 to D28, D33 to D29, D34 to D30, D36 to D31, D37 to D32, D38 to D33, D39 to D34, D40 to D35, D41 to D36, D43 to D37, D44 to D38, D45 to D39, D46 to D40, D47 to D41, D48 to D42, D50 to D43, D51 to D44, D52 to D45, D53 to D46, D54 to D47, D55 to D48, D8 to D7, D9 to D8, D10 to D9, SW11 to SW10, SW12 to SW11, SW13 to SW12, SW15 to SW13, SW16 to SW14, SW17 to SW15, SW18 to SW16, SW19 to SW17, SW20 to SW18, SW22 to SW19, SW23 to SW20, SW24 to SW21, SW25 to SW22, SW26 to SW23, SW27 to SW24, SW29 to SW25, SW30 to SW26, SW31 to SW27, SW32 to SW28, SW33 to SW29, SW34 to SW30, SW36 to SW31, SW37 to SW32, SW38 to SW33, SW39 to SW34, SW40 to SW35, SW41 to SW36, SW43 to SW37, SW44 to SW38, SW45 to SW39, SW46 to SW40, SW47 to SW41, SW48 to SW42, SW50 to SW43, SW51 to SW44, SW52 to SW45, SW53 to SW46, SW54 to SW47, SW55 to SW48, SW8 to SW7, SW9 to SW8, SW10 to SW9
Connections:
- net ROW0: now also D49.1 (K), U1.10 (GP9); no longer U1.9 (GP8)
- net ROW1: now also U1.11 (GP10), D50.1 (K); no longer U1.10 (GP9)
- net ROW2: now also U1.12 (GP11), D51.1 (K); no longer U1.11 (GP10)
- net ROW3: now also U1.13 (GP12), D52.1 (K); no longer U1.12 (GP11)
- net ROW4: now also U1.14 (GP13), D53.1 (K); no longer U1.13 (GP12)
- net ROW5: now also U1.15 (GP14), D54.1 (K); no longer U1.14 (GP13)
- net at U1.17 (GP26): now also SW55.A
- net at U1.18 (GP27): now also SW55.B
- net at U1.19 (GP28): now also CN1.4
- net at U1.20 (GP29): now also CN1.3
- net at U1.22 (GND): now also CN1.5, SW55.C
- net at U1.23 (5V): now also CN1.2
- net BTN2: now reaches D49.2 (A)
- net BTN2: now also SW55.E
- removed net ROW6: D49.1 (K), U1.15 (GP14)
- new net: D50.2 (A), SW50.2
- new net: D54.2 (A), SW54.2
- new net: D53.2 (A), SW53.2
- new net: D51.2 (A), SW51.2
- new net: D52.2 (A), SW52.2
- new net BTN1: SW50.1, SW51.1, SW52.1, SW53.1, SW54.1, SW55.D, U1.9 (GP8)
- no-connect marks 4 -> 2
Other:
- moved on the sheet: D1, D10, D11, D12, D13, D14, D15, D16, D17, D18, D19, D2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
